File: _autosave-45-pcb.kicad_pcb (KiCad board)
At the start: 2 copper layers, 1.6 x 38.1 mm, 24 parts, among them SW1 SW_Push, U1 ATmega32U4-AU, Y1 16MHz

Commit message: Traces Finished
PCB done
Parts:
- F1, SW1: moved to B.Cu
- moved SW1 86.5 mm to (67.5, 142.9), turned to 180 degrees
- moved F1 61.3 mm to (60.5, 121.9), turned to 90 degrees
- moved R4 49.6 mm to (100.8, 134.3), turned to 90 degrees
- moved D3 27.0 mm to (140.6, 118.2)
- moved D2 26.9 mm to (121.5, 137.3)
- moved R2 22.6 mm to (70.9, 119.8), turned to 90 degrees
- moved R1 22.2 mm to (66.3, 119.8), turned to 90 degrees
- moved C3 1.32 mm to (83.9, 121.1)
- moved C1 1.10 mm to (101.5, 126.3)
- moved R3 0.69 mm to (80.0, 121.7), turned to 270 degrees
Routing:
- net GND: track 0.00 -> 149.6 mm, vias 0 -> 2
- net +5V: track 0.00 -> 110.5 mm, vias 0 -> 4
- net Net-(R3-Pad2): track 0.00 -> 36.8 mm, vias 0 -> 4
- net Net-(R1-Pad1): track 0.00 -> 28.2 mm
- net Net-(R2-Pad1): track 0.00 -> 26.4 mm
- net ROW0: track 0.00 -> 20.5 mm
- net ROW1: track 0.00 -> 20.4 mm
- net COL1: track 0.00 -> 18.1 mm
- net COL0: track 0.00 -> 18.1 mm
- net Net-(C5-Pad1): track 0.00 -> 13.1 mm
- net VCC: track 0.00 -> 10.7 mm
- net Net-(C4-Pad1): track 0.00 -> 9.49 mm
- net Net-(C7-Pad1): track 0.00 -> 7.85 mm, vias 0 -> 2
- net Net-(D3-Pad2): track 0.00 -> 6.70 mm
- net Net-(D2-Pad2): track 0.00 -> 6.70 mm
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Other:
- board size 1.6 x 38.1 mm -> 84.1 x 38.1 mm
- net class Default: trace_width 0.25 -> 0.254
- net class Power added: clearance 0.2, trace_width 0.381, via_dia 0.8, via_drill 0.4

Commit message: Done
Parts:
- renumbered D3 to D2, D2 to D3
Connections:
- U1 pad 27: Net-(U1-Pad27) -> ROW0
- U1 pad 28: Net-(U1-Pad28) -> COL1
- U1 pad 29: Net-(U1-Pad29) -> COL0
- U1 pad 30: Net-(U1-Pad30) -> ROW1
Routing:
- net COL1: track 18.1 -> 53.4 mm, vias 0 -> 3
- net ROW1: track 20.4 -> 53.3 mm, vias 0 -> 2
- net ROW0: track 20.5 -> 48.6 mm, vias 0 -> 2
- net COL0: track 18.1 -> 31.1 mm, vias 0 -> 1
