File: 45-pcb.kicad_pcb (KiCad board)
At the start: 2 copper layers, 84.1 x 38.1 mm, 24 parts, among them SW1 SW_Push, U1 ATmega32U4-AU, Y1 16MHz

Commit message: Done
Parts:
- moved D2 27.0 mm to (140.6, 118.2)
- moved D3 26.9 mm to (121.5, 137.3)
- moved F1 3.68 mm to (60.5, 121.9), turned to 90 degrees
- moved C3 1.32 mm to (83.9, 121.1)
- moved C1 1.10 mm to (101.5, 126.3)
- moved R3 0.69 mm to (80.0, 121.7), turned to 270 degrees
- renumbered D3 to D2, D2 to D3
Connections:
- U1 pad 27: Net-(U1-Pad27) -> ROW0
- U1 pad 28: Net-(U1-Pad28) -> COL1
- U1 pad 29: Net-(U1-Pad29) -> COL0
- U1 pad 30: Net-(U1-Pad30) -> ROW1
Routing:
- net GND: track 0.00 -> 149.6 mm, vias 0 -> 2
- net +5V: track 0.00 -> 110.5 mm, vias 0 -> 4
- net ROW1: track 0.00 -> 53.3 mm, vias 0 -> 2
- net COL1: track 0.00 -> 50.9 mm, vias 0 -> 3
- net ROW0: track 0.00 -> 48.6 mm, vias 0 -> 2
- net Net-(R3-Pad2): track 0.00 -> 36.8 mm, vias 0 -> 4
- net COL0: track 0.00 -> 31.1 mm, vias 0 -> 1
- net Net-(R1-Pad1): track 0.00 -> 28.2 mm
- net Net-(R2-Pad1): track 0.00 -> 26.4 mm
- net Net-(C5-Pad1): track 0.00 -> 13.1 mm
- net VCC: track 0.00 -> 10.7 mm
- net Net-(C4-Pad1): track 0.00 -> 9.49 mm
- net Net-(C7-Pad1): track 0.00 -> 7.85 mm, vias 0 -> 2
- net Net-(D2-Pad2): track 0.00 -> 6.90 mm
- net Net-(D3-Pad2): track 0.00 -> 6.90 mm
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- added copper zone on B.Cu, net GND
Other:
- board text added: "Guide"
