File: 45-pcb.sch (KiCad schematic (older format))
At the start: 24 parts, among them SW1 SW_Push, U1 ATmega32U4-AU, Y1 16MHz

Commit message: Done
Parts:
- renumbered D3 to D2, D2 to D3
Connections:
- net COL0: now also U1.29 (PB5)
- net COL1: now also U1.28 (PB4)
- net ROW0: now also U1.27 (PD7)
- net ROW1: now also U1.30 (PB6)
Changed lines of the file:
@@
 $EndComp
 $Comp
-L Device:D_Small D3
+L Device:D_Small D2
 U 1 1 5EF62358
 P 7550 1600
-F 0 "D3" V 7596 1530 50  0000 R CNN
+F 0 "D2" V 7596 1530 50  0000 R CNN
 F 1 "D_Small" V 7505 1530 50  0000 R CNN
 F 2 "Diode_SMD:D_SOD-123" V 7550 1600 50  0001 C CNN
@@
 	6600 2350 6900 2350
 $Comp
-L Device:D_Small D2
+L Device:D_Small D3
 U 1 1 5EF8251B
 P 6900 2250
-F 0 "D2" V 6946 2180 50  0000 R CNN
+F 0 "D3" V 6946 2180 50  0000 R CNN
 F 1 "D_Small" V 6855 2180 50  0000 R CNN
 F 2 "Diode_SMD:D_SOD-123" V 6900 2250 50  0001 C CNN
@@
 Wire Wire Line
 	6900 2350 7550 2350
+Text GLabel 5000 3150 2    50   Input ~ 0
+COL1
+Text GLabel 5000 3250 2    50   Input ~ 0
+COL0
+Text GLabel 5000 3350 2    50   Input ~ 0
+ROW1
+Text GLabel 5000 4650 2    50   Input ~ 0
+ROW0
 $EndSCHEMATC
